File: holder.kicad_pcb (KiCad board)
At the start: 2 copper layers, 58 x 88 mm, 24 parts

Commit message: ...
Parts:
- added SOT-223: SOT-223, Package_TO_SOT_SMD:SOT-223, F.Cu at (204.0, 137.5)
- renumbered REF** to 6x6mm, LFBGA-144 to LFBGA-144/0.8mm, LGA-16 to LGA-16/0.5mm, LGA-8 to LGA-8/0.65mm, LQFP-32 to LQFP-32/0.8mm, LQFP-48 to LQFP-48/0.5mm, LQFP-64 to LQFP-64/0.5mm, SOP-8 to SOP-8/1.27mm, TSSOP-20 to TSSOP-20/0.65mm
Routing:
- net (no net): track 0.00 -> 36.0 mm
Other:
- outline, holes or cut-outs redrawn
- board text added: "A"
- board text added: "B"
- board text added: "Bipolar NPN"
- board text added: "C"
- board text added: "Capacitor"
- board text added: "Coil"
- board text added: "D"
- board text added: "Diode"
- board text added: "E"
- board text added: "Frequency f[Hz] = n/t[s] T[s] = 1/f[Hz]"
- board text added: "G"
- board text added: "N-MOSFET"
- board text added: "Resistor"
- board text added: "S"
- board text added: "Tracks 0,25mm 0,3mm 0,5mm 0,8mm 1mm 1,2mm 1,5mm 2mm"
- board text added: "Wavelength λ[m] = c/f[Hz] c = 299'792'458 m/s"
- board text removed: "Wavelength λ = c/f[Hz] c = 299'792'458 m/s"

Commit message: added field
Routing:
- added copper zone on B.Cu, net (none)
Changed lines of the file:
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@@
   )
   (setup
-    (last_trace_width 2)
+    (last_trace_width 0.25)
     (user_trace_width 0.3)
     (user_trace_width 0.5)
@@
   (segment (start 197.5 87) (end 202 87) (width 1.5) (layer F.Cu) (net 0))
   (segment (start 197.5 89) (end 202 89) (width 2) (layer F.Cu) (net 0))
+  (zone (net 0) (net_name "") (layer B.Cu) (hatch edge 0.508)
+    (connect_pads (clearance 0.508))
+    (min_thickness 0.254)
+    (fill yes (arc_segments 32) (thermal_gap 0.508) (thermal_bridge_width 0.508))
+    (polygon
+      (pts
+        (xy 160 60) (xy 160 148) (xy 218 148) (xy 218 60)
+      )
+    )
+  )
 )
